File: PowerWheelzSchematics/batteryLayout.sch (KiCad schematic (older format))
At the start: 25 parts

Commit message: Name added
Parts:
- U? (x25): symbol VESE:18650 -> PowerWheelzSchematics-rescue:18650-VESE
Changed lines of the file:
@@
 Comp "VESE"
 Comment1 "Alex Domagala"
-Comment2 ""
+Comment2 "Jonathan Perthel"
 Comment3 ""
 Comment4 ""
@@
 5S5P Layout (5 Cells Series, 5 Cells Parallel)\n
 $Comp
-L VESE:18650 U?
+L PowerWheelzSchematics-rescue:18650-VESE U?
 U 1 1 5F86A33D
 P 2475 2000
+AR Path="/5F86A33D" Ref="U?"  Part="1"
+AR Path="/5F8680B4/5F86A33D" Ref="U?"  Part="1"
 F 0 "U?" H 2653 1821 50  0001 L CNN
 F 1 "18650" H 2653 1775 50  0001 L CNN
@@
 $EndComp
 $Comp
-L VESE:18650 U?
+L PowerWheelzSchematics-rescue:18650-VESE U?
 U 1 1 5F86C075
 P 2975 2000
+AR Path="/5F86C075" Ref="U?"  Part="1"
+AR Path="/5F8680B4/5F86C075" Ref="U?"  Part="1"
 F 0 "U?" H 3153 1821 50  0001 L CNN
 F 1 "18650" H 3153 1775 50  0001 L CNN
@@
 $EndComp
 $Comp
-L VESE:18650 U?
+L PowerWheelzSchematics-rescue:18650-VESE U?
 U 1 1 5F8715AC
 P 3425 2000
+AR Path="/5F8715AC" Ref="U?"  Part="1"
+AR Path="/5F8680B4/5F8715AC" Ref="U?"  Part="1"
 F 0 "U?" H 3603 1821 50  0001 L CNN
 F 1 "18650" H 3603 1775 50  0001 L CNN
@@
 $EndComp
 $Comp
-L VESE:18650 U?
+L PowerWheelzSchematics-rescue:18650-VESE U?
 U 1 1 5F8715B2
 P 3925 2000
+AR Path="/5F8715B2" Ref="U?"  Part="1"
+AR Path="/5F8680B4/5F8715B2" Ref="U?"  Part="1"
 F 0 "U?" H 4103 1821 50  0001 L CNN
 F 1 "18650" H 4103 1775 50  0001 L CNN
@@
 $EndComp
 $Comp
-L VESE:18650 U?
+L PowerWheelzSchematics-rescue:18650-VESE U?
 U 1 1 5F881C08
 P 4425 2000
+AR Path="/5F881C08" Ref="U?"  Part="1"
+AR Path="/5F8680B4/5F881C08" Ref="U?"  Part="1"
 F 0 "U?" H 4603 1821 50  0001 L CNN
 F 1 "18650" H 4603 1775 50  0001 L CNN
@@
 	4000 2700 4500 2700
 $Comp
-L VESE:18650 U?
+L PowerWheelzSchematics-rescue:18650-VESE U?
 U 1 1 5F8DC48E
 P 2475 2950
+AR Path="/5F8DC48E" Ref="U?"  Part="1"
+AR Path="/5F8680B4/5F8DC48E" Ref="U?"  Part="1"
 F 0 "U?" H 2653 2771 50  0001 L CNN
 F 1 "18650" H 2653 2725 50  0001 L CNN
@@
 $EndComp
 $Comp
-L VESE:18650 U?
+L PowerWheelzSchematics-rescue:18650-VESE U?
 U 1 1 5F8DC494
 P 2975 2950
+AR Path="/5F8DC494" Ref="U?"  Part="1"
+AR Path="/5F8680B4/5F8DC494" Ref="U?"  Part="1"
 F 0 "U?" H 3153 2771 50  0001 L CNN
 F 1 "18650" H 3153 2725 50  0001 L CNN
@@
 $EndComp
 $Comp
-L VESE:18650 U?
+L PowerWheelzSchematics-rescue:18650-VESE U?
 U 1 1 5F8DC49A
 P 3425 2950
+AR Path="/5F8DC49A" Ref="U?"  Part="1"
+AR Path="/5F8680B4/5F8DC49A" Ref="U?"  Part="1"
 F 0 "U?" H 3603 2771 50  0001 L CNN
 F 1 "18650" H 3603 2725 50  0001 L CNN
@@
 $EndComp
 $Comp
-L VESE:18650 U?
+L PowerWheelzSchematics-rescue:18650-VESE U?
 U 1 1 5F8DC4A0
 P 3925 2950
+AR Path="/5F8DC4A0" Ref="U?"  Part="1"
+AR Path="/5F8680B4/5F8DC4A0" Ref="U?"  Part="1"
 F 0 "U?" H 4103 2771 50  0001 L CNN
 F 1 "18650" H 4103 2725 50  0001 L CNN
@@
 $EndComp
 $Comp
-L VESE:18650 U?
+L PowerWheelzSchematics-rescue:18650-VESE U?
 U 1 1 5F8DC4A6
 P 4425 2950
+AR Path="/5F8DC4A6" Ref="U?"  Part="1"
+AR Path="/5F8680B4/5F8DC4A6" Ref="U?"  Part="1"
 F 0 "U?" H 4603 2771 50  0001 L CNN
 F 1 "18650" H 4603 2725 50  0001 L CNN
@@
 	4000 3650 4500 3650
 $Comp
-L VESE:18650 U?
+L PowerWheelzSchematics-rescue:18650-VESE U?
 U 1 1 5F8E1749
 P 2475 3900
+AR Path="/5F8E1749" Ref="U?"  Part="1"
+AR Path="/5F8680B4/5F8E1749" Ref="U?"  Part="1"
 F 0 "U?" H 2653 3721 50  0001 L CNN
 F 1 "18650" H 2653 3675 50  0001 L CNN
@@
 $EndComp
 $Comp
-L VESE:18650 U?
+L PowerWheelzSchematics-rescue:18650-VESE U?
 U 1 1 5F8E174F
 P 2975 3900
+AR Path="/5F8E174F" Ref="U?"  Part="1"
+AR Path="/5F8680B4/5F8E174F" Ref="U?"  Part="1"
 F 0 "U?" H 3153 3721 50  0001 L CNN
 F 1 "18650" H 3153 3675 50  0001 L CNN
@@
 $EndComp
 $Comp
-L VESE:18650 U?
+L PowerWheelzSchematics-rescue:18650-VESE U?
 U 1 1 5F8E1755
 P 3425 3900
+AR Path="/5F8E1755" Ref="U?"  Part="1"
+AR Path="/5F8680B4/5F8E1755" Ref="U?"  Part="1"
 F 0 "U?" H 3603 3721 50  0001 L CNN
 F 1 "18650" H 3603 3675 50  0001 L CNN
@@
 $EndComp
 $Comp
-L VESE:18650 U?
+L PowerWheelzSchematics-rescue:18650-VESE U?
 U 1 1 5F8E175B
 P 3925 3900
+AR Path="/5F8E175B" Ref="U?"  Part="1"
+AR Path="/5F8680B4/5F8E175B" Ref="U?"  Part="1"
 F 0 "U?" H 4103 3721 50  0001 L CNN
 F 1 "18650" H 4103 3675 50  0001 L CNN
@@
 $EndComp
 $Comp
-L VESE:18650 U?
+L PowerWheelzSchematics-rescue:18650-VESE U?
 U 1 1 5F8E1761
 P 4425 3900
+AR Path="/5F8E1761" Ref="U?"  Part="1"
+AR Path="/5F8680B4/5F8E1761" Ref="U?"  Part="1"
 F 0 "U?" H 4603 3721 50  0001 L CNN
 F 1 "18650" H 4603 3675 50  0001 L CNN
@@
 	4000 4600 4500 4600
 $Comp
-L VESE:18650 U?
+L PowerWheelzSchematics-rescue:18650-VESE U?
 U 1 1 5F8E6FBF
 P 2475 4850
+AR Path="/5F8E6FBF" Ref="U?"  Part="1"
+AR Path="/5F8680B4/5F8E6FBF" Ref="U?"  Part="1"
 F 0 "U?" H 2653 4671 50  0001 L CNN
 F 1 "18650" H 2653 4625 50  0001 L CNN
@@
 $EndComp
 $Comp
-L VESE:18650 U?
+L PowerWheelzSchematics-rescue:18650-VESE U?
 U 1 1 5F8E6FC5
 P 2975 4850
+AR Path="/5F8E6FC5" Ref="U?"  Part="1"
+AR Path="/5F8680B4/5F8E6FC5" Ref="U?"  Part="1"
 F 0 "U?" H 3153 4671 50  0001 L CNN
 F 1 "18650" H 3153 4625 50  0001 L CNN
@@
 $EndComp
 $Comp
-L VESE:18650 U?
+L PowerWheelzSchematics-rescue:18650-VESE U?
 U 1 1 5F8E6FCB
 P 3425 4850
+AR Path="/5F8E6FCB" Ref="U?"  Part="1"
+AR Path="/5F8680B4/5F8E6FCB" Ref="U?"  Part="1"
 F 0 "U?" H 3603 4671 50  0001 L CNN
 F 1 "18650" H 3603 4625 50  0001 L CNN
@@
 $EndComp
 $Comp
-L VESE:18650 U?
+L PowerWheelzSchematics-rescue:18650-VESE U?
 U 1 1 5F8E6FD1
 P 3925 4850
+AR Path="/5F8E6FD1" Ref="U?"  Part="1"
+AR Path="/5F8680B4/5F8E6FD1" Ref="U?"  Part="1"
 F 0 "U?" H 4103 4671 50  0001 L CNN
 F 1 "18650" H 4103 4625 50  0001 L CNN
@@
 $EndComp
 $Comp
-L VESE:18650 U?
+L PowerWheelzSchematics-rescue:18650-VESE U?
 U 1 1 5F8E6FD7
 P 4425 4850
+AR Path="/5F8E6FD7" Ref="U?"  Part="1"
+AR Path="/5F8680B4/5F8E6FD7" Ref="U?"  Part="1"
 F 0 "U?" H 4603 4671 50  0001 L CNN
 F 1 "18650" H 4603 4625 50  0001 L CNN
@@
 Connection ~ 4500 4600
 $Comp
-L VESE:18650 U?
+L PowerWheelzSchematics-rescue:18650-VESE U?
 U 1 1 5F93CCE0
 P 2475 5800
+AR Path="/5F93CCE0" Ref="U?"  Part="1"
+AR Path="/5F8680B4/5F93CCE0" Ref="U?"  Part="1"
 F 0 "U?" H 2653 5621 50  0001 L CNN
 F 1 "18650" H 2653 5575 50  0001 L CNN
@@
 $EndComp
 $Comp
-L VESE:18650 U?
+L PowerWheelzSchematics-rescue:18650-VESE U?
 U 1 1 5F93CCE6
 P 2975 5800
+AR Path="/5F93CCE6" Ref="U?"  Part="1"
+AR Path="/5F8680B4/5F93CCE6" Ref="U?"  Part="1"
 F 0 "U?" H 3153 5621 50  0001 L CNN
 F 1 "18650" H 3153 5575 50  0001 L CNN
@@
 $EndComp
 $Comp
-L VESE:18650 U?
+L PowerWheelzSchematics-rescue:18650-VESE U?
 U 1 1 5F93CCEC
 P 3425 5800
+AR Path="/5F93CCEC" Ref="U?"  Part="1"
+AR Path="/5F8680B4/5F93CCEC" Ref="U?"  Part="1"
 F 0 "U?" H 3603 5621 50  0001 L CNN
 F 1 "18650" H 3603 5575 50  0001 L CNN
@@
 $EndComp
 $Comp
-L VESE:18650 U?
+L PowerWheelzSchematics-rescue:18650-VESE U?
 U 1 1 5F93CCF2
 P 3925 5800
+AR Path="/5F93CCF2" Ref="U?"  Part="1"
+AR Path="/5F8680B4/5F93CCF2" Ref="U?"  Part="1"
 F 0 "U?" H 4103 5621 50  0001 L CNN
 F 1 "18650" H 4103 5575 50  0001 L CNN
@@
 $EndComp
 $Comp
-L VESE:18650 U?
+L PowerWheelzSchematics-rescue:18650-VESE U?
 U 1 1 5F93CCF8
 P 4425 5800
+AR Path="/5F93CCF8" Ref="U?"  Part="1"
+AR Path="/5F8680B4/5F93CCF8" Ref="U?"  Part="1"
 F 0 "U?" H 4603 5621 50  0001 L CNN
 F 1 "18650" H 4603 5575 50  0001 L CNN
