File: PowerWheelzSchematics/batteryLayout5S5P.sch (KiCad schematic (older format))
At the start: 25 parts

Commit message: 5S5P update
Parts:
- added U?: BMS, symbol VESE:BMS
Connections:
- wire segments 80 -> 95
- no-connect marks 2 -> 1
Changed lines of the file:
@@
 	3700 4450 3950 4450
-Wire Wire Line
-	3700 2500 3700 3000
 Wire Wire Line
 	3950 2500 3700 2500
@@
 	7500 4450 7250 4450
 Wire Wire Line
-	7250 2500 7500 2500
+	7250 2500 7425 2500
 $Comp
 L PowerWheelzSchematics-rescue:18650-VESE U?
@@
 	0    1    1    0
 $EndComp
-Wire Wire Line
-	7500 4450 7500 4750
-Wire Wire Line
-	7500 4750 5250 4750
-Wire Wire Line
-	5250 4750 5250 5000
+$Comp
+L VESE:BMS U?
+U 1 1 5F954BBE
+P 6750 1275
+F 0 "U?" H 6825 1200 50  0001 C CNN
+F 1 "BMS" H 7178 1358 50  0000 C CNN
+F 2 "" H 6825 1200 50  0001 C CNN
+F 3 "" H 6825 1200 50  0001 C CNN
+	1    6750 1275
+	1    0    0    -1
+$EndComp
+Wire Wire Line
+	6800 2125 2750 2125
+Wire Wire Line
+	2750 2125 2750 2500
+Connection ~ 2750 2500
+Wire Wire Line
+	6925 2175 3700 2175
+Wire Wire Line
+	3700 2175 3700 2500
+Wire Wire Line
+	6925 2125 6925 2175
+Wire Wire Line
+	7050 2125 7050 2225
+Wire Wire Line
+	7050 2225 4650 2225
+Wire Wire Line
+	4650 2225 4650 2500
+Wire Wire Line
+	3700 2500 3700 3000
+Wire Wire Line
+	7175 2125 7175 2275
+Wire Wire Line
+	7175 2275 5600 2275
+Wire Wire Line
+	5600 2275 5600 2500
+Wire Wire Line
+	7300 2125 7300 2325
+Wire Wire Line
+	7300 2325 6550 2325
+Wire Wire Line
+	6550 2325 6550 2500
+Wire Wire Line
+	7425 2125 7425 2500
+Connection ~ 7425 2500
+Wire Wire Line
+	7425 2500 7500 2500
+Wire Wire Line
+	7500 4450 9250 4450
 Connection ~ 7500 4450
-Wire Wire Line
-	2750 4450 2750 4750
-Wire Wire Line
-	2750 4750 5000 4750
-Wire Wire Line
-	5000 4750 5000 5000
+NoConn ~ 9250 4450
+Wire Wire Line
+	7600 1525 7750 1525
+Wire Wire Line
+	7750 1525 7750 4625
+Wire Wire Line
+	7750 4625 2750 4625
+Wire Wire Line
+	2750 4625 2750 4450
 Connection ~ 2750 4450
-NoConn ~ 5000 5000
-NoConn ~ 5250 5000
 $EndSCHEMATC

Commit message: Added Load & Supply
Parts:
- added U?: Load, symbol PowerWheelzSchematics-rescue:Load
- added U?: Supply, symbol PowerWheelzSchematics-rescue:Supply
- U?: symbol VESE:BMS -> PowerWheelzSchematics-rescue:BMS-VESE
Connections:
- wire segments 95 -> 107
Other:
- note added: "The B- Terminal is the net negative terminal for the entire battery"
- note added: "The C- wire connects to the negative terminal for the Charge (supply)"
- note added: "The GND pin connects to the negative terminal of the first battery in series\n"
- note added: "The P- wire connects to the negative terminal of the load\n"
- note added: "The Supply represents a connection to Power Supply\n"
- note added: "The load represents the connection to motor"
- note added: "This is + wire conneceting to Load and supply\n"
- note added: "This is the Balanced Inputs which connects to the positive terminal to each battery in series"
Changed lines of the file:
@@
 $EndComp
 $Comp
-L VESE:BMS U?
+L PowerWheelzSchematics-rescue:BMS-VESE U?
 U 1 1 5F954BBE
 P 6750 1275
+AR Path="/5F954BBE" Ref="U?"  Part="1"
+AR Path="/5F8680B4/5F954BBE" Ref="U?"  Part="1"
 F 0 "U?" H 6825 1200 50  0001 C CNN
 F 1 "BMS" H 7178 1358 50  0000 C CNN
@@
 	7425 2500 7500 2500
 Wire Wire Line
-	7500 4450 9250 4450
+	7500 4450 8400 4450
 Connection ~ 7500 4450
 NoConn ~ 9250 4450
@@
 	2750 4625 2750 4450
 Connection ~ 2750 4450
+$Comp
+L PowerWheelzSchematics-rescue:Load U?
+U 1 1 5F952371
+P 8200 3950
+F 0 "U?" H 8300 3900 50  0001 C CNN
+F 1 "Load" H 8628 3850 39  0000 L CNN
+F 2 "" H 8300 3900 50  0001 C CNN
+F 3 "" H 8300 3900 50  0001 C CNN
+	1    8200 3950
+	1    0    0    -1
+$EndComp
+Wire Wire Line
+	7600 1450 7600 1425
+Connection ~ 7600 1425
+Wire Wire Line
+	7600 1425 7600 1400
+$Comp
+L PowerWheelzSchematics-rescue:Supply U?
+U 1 1 5F962F29
+P 9000 3950
+F 0 "U?" H 9150 3900 50  0001 C CNN
+F 1 "Supply" H 9328 3875 50  0000 L CNN
+F 2 "" H 9150 3900 50  0001 C CNN
+F 3 "" H 9150 3900 50  0001 C CNN
+	1    9000 3950
+	1    0    0    -1
+$EndComp
+Wire Wire Line
+	9150 4200 9150 4450
+Connection ~ 9150 4450
+Wire Wire Line
+	9150 4450 9250 4450
+Wire Wire Line
+	8400 4250 8400 4450
+Connection ~ 8400 4450
+Wire Wire Line
+	8400 4450 9150 4450
+Wire Wire Line
+	8400 3850 8400 1400
+Wire Wire Line
+	8400 1400 7600 1400
+Wire Wire Line
+	9150 3850 9150 1300
+Wire Wire Line
+	9150 1300 7600 1300
+Wire Wire Line
+	7600 1300 7600 1325
+Connection ~ 7600 1325
+Wire Wire Line
+	7600 1325 7600 1350
+Text Notes 2950 1850 0    50   ~ 0
+This is the Balanced Inputs which connects to the positive terminal to each battery in series
+Text Notes 7850 4650 0    50   ~ 0
+This is + wire conneceting to Load and supply\n
+Text Notes 7600 950  0    50   ~ 0
+The C- wire connects to the negative terminal for the Charge (supply)
+Text Notes 7600 1050 0    50   ~ 0
+The P- wire connects to the negative terminal of the load\n
+Text Notes 7600 1150 0    50   ~ 0
+The B- Terminal is the net negative terminal for the entire battery
+Text Notes 9200 3450 0    50   ~ 0
+The load represents the connection to motor
+Text Notes 9200 3600 0    50   ~ 0
+The Supply represents a connection to Power Supply\n
+Text Notes 2950 2000 0    50   ~ 0
+The GND pin connects to the negative terminal of the first battery in series\n
 $EndSCHEMATC

Commit message: Fixes
Connections:
- wire segments 107 -> 104

Commit message: Big Update
Connections:
- wire segments 104 -> 103
- no-connect marks 1 -> 0
Other:
- note added: "+V wire conneceting to Load and Supply\n"
- note added: "0V"
- note added: "10.8V"
- note added: "14.4V"
- note added: "18.0V"
- note added: "3.6V"
- note added: "7.2V"
- note added: "B- terminal is the net negative terminal for the entire battery"
- note added: "Balance Inputs: connect to the positive terminals of each battery in series"
- note added: "C- connects to the negative terminal for the Charge"
- note added: "GND: connects to the negative terminal of the first battery in series\n"
- note added: "P- wire connects to the negative terminal for the Load\n"
- note added: "The Load represents the connection to Motor"
- note added: "The Supply represents a connection to Charger\n"
- note added: "XT90"
- note removed: "The B- Terminal is the net negative terminal for the entire battery"
- note removed: "The C- wire connects to the negative terminal for the Charge (supply)"
- note removed: "The GND pin connects to the negative terminal of the first battery in series\n"
- note removed: "The P- wire connects to the negative terminal of the load\n"
- note removed: "The Supply represents a connection to Power Supply\n"
- note removed: "The load represents the connection to motor"
- note removed: "This is + wire conneceting to Load and supply\n"
- note removed: "This is the Balanced Inputs which connects to the positive terminal to each battery in series"
Changed lines of the file:
@@
 $Descr A4 11693 8268
 encoding utf-8
-Sheet 2 3
+Sheet 3 3
 Title "Battery Layout"
 Date "2020-10-13"
@@
 Wire Wire Line
 	5800 2975 5800 3150
-NoConn ~ 8350 5100
 Wire Wire Line
 	6850 2175 7000 2175
@@
 	7400 4500 7400 2075
 Text Notes 2200 2500 0    50   ~ 0
-This is the Balanced Inputs which connects to the positive terminal to each battery in series
+Balance Inputs: connect to the positive terminals of each battery in series
 Text Notes 7075 5250 0    50   ~ 0
-This is + wire conneceting to Load and supply\n
++V wire conneceting to Load and Supply\n
 Text Notes 6850 1600 0    50   ~ 0
-The C- wire connects to the negative terminal for the Charge (supply)
+C- connects to the negative terminal for the Charge
 Text Notes 6850 1700 0    50   ~ 0
-The P- wire connects to the negative terminal of the load\n
+P- wire connects to the negative terminal for the Load\n
 Text Notes 6850 1800 0    50   ~ 0
-The B- Terminal is the net negative terminal for the entire battery
+B- terminal is the net negative terminal for the entire battery
 Text Notes 8550 4675 0    50   ~ 0
-The load represents the connection to motor
+The Load represents the connection to Motor
 Text Notes 8550 4825 0    50   ~ 0
-The Supply represents a connection to Power Supply\n
+The Supply represents a connection to Charger\n
 Text Notes 2200 2650 0    50   ~ 0
-The GND pin connects to the negative terminal of the first battery in series\n
+GND: connects to the negative terminal of the first battery in series\n
 Wire Wire Line
 	6500 3150 6750 3150
@@
 	7400 5100 8000 5100
 Connection ~ 7400 5100
-Wire Wire Line
-	8000 5100 8350 5100
-Connection ~ 8000 5100
+Text Notes 7325 4725 0    39   ~ 0
+XT90
+Text Notes 2075 5175 0    50   ~ 0
+0V
+Text Notes 2875 5200 0    50   ~ 0
+3.6V
+Text Notes 3825 5200 0    50   ~ 0
+7.2V
+Text Notes 4750 5200 0    50   ~ 0
+10.8V
+Text Notes 5725 5200 0    50   ~ 0
+14.4V
+Text Notes 6650 5200 0    50   ~ 0
+18.0V
 $EndSCHEMATC
